Commit message: Transfer to shadow hand
Commented world link in URDF

File: hand_embodiment/model/sr_common/sr_description/urdf/shadow_hand.urdf (robot description, URDF)
Before this commit: robot shadowhand_motor, 33 links, 32 joints
Links:
- removed link world
Joints:
- removed joint rh_world_joint
