Commit message: Switch back to default Mia hand URDF

File: hand_embodiment/model/mia_hand_ros_pkgs/mia_hand_description/urdf/mia_hand.urdf.xacro (robot description, xacro)
@@ -1,366 +1,383 @@
-<?xml version="1.0"?>
+<?xml version="1.0" ?>
+<!-- =================================================================================== -->
+<!-- |    This document was autogenerated by xacro from mia_hand.urdf.xacro            | -->
+<!-- |    EDITING THIS FILE BY HAND IS NOT RECOMMENDED                                 | -->
+<!-- =================================================================================== -->
 <!-- created with Phobos 1.0.1 "Capricious Choutengan" -->
-  <!-- model version="4.4.1"-->
-  <robot xmlns:xacro="http://wiki.ros.org/xacro" name="mia_hand"
-  xmlns:sensor="http://playerstage.sourceforge.net/gazebo/xmlschema/#sensor"
-  xmlns:controller="http://playerstage.sourceforge.net/gazebo/xmlschema/#controller"
-  xmlns:joint="http://playerstage.sourceforge.net/gazebo/xmlschema/#slider"
-  xmlns:interface="http://playerstage.sourceforge.net/gazebo/xmlschema/#interface"
-  xmlns:body="http://playerstage.sourceforge.net/gazebo/xmlschema/#body"
-  xmlns:geom="http://playerstage.sourceforge.net/gazebo/xmlschema/#geom">
-    <link name="index_fle">
-      <inertial>
-        <origin xyz="-0.000420165 0.007306039 0.000122778" rpy="0 0 0"/>
-        <mass value="0.0113"/>
-        <inertia ixx="1.486e-06" ixy="0" ixz="0" iyy="2e-07" iyz="0" izz="8.31e-07"/>
-      </inertial>
-      <collision name="collision_index_pre_sensor">
-        <origin xyz="0.000159719 0.023606986 0.001508433" rpy="1.611356378 -1.479902387 -0.009164433"/>
-        <geometry>
-          <cylinder radius="0.007128498" length="0.016970539"/>
-        </geometry>
-      </collision>
-    </link>
-    <link name="index_sensor">
-      <inertial>
-        <origin xyz="0.000343341 0.026805416 0.000475764" rpy="0 0 0"/>
-        <mass value="0.0132"/>
-        <inertia ixx="4.063e-06" ixy="9.32e-07" ixz="0" iyy="1.01e-06" iyz="-5e-09" izz="4.81e-06"/>
-      </inertial>
-      <visual >
-        <origin xyz="-0.016737008 -0.126896188 -0.051269896" rpy="0.457628608 -1.375251532 0.776470125"/>
-        <geometry>
-          <mesh filename="package://mia_hand_description/meshes/stl/index_finger.stl" scale="0.000999987 0.000999987 0.000999987"/>
-        </geometry>
-        <material name="BLACK"/>
-      </visual>
-      <visual >
-        <origin xyz="-0.016737008 -0.126896188 -0.051269896" rpy="0.457628608 -1.375251532 0.776470125"/>
-        <geometry>
-          <mesh filename="package://mia_hand_description/meshes/stl/index_tip.stl" scale="0.000999987 0.000999987 0.000999987"/>
-        </geometry>
-        <material name="WHITE"/>
-      </visual>
-      <collision name="collision_index_distal">
-        <origin xyz="-0.001899783 0.0412638 0.001381427" rpy="1.826135755 -1.502358675 0.115027599"/>
-        <geometry>
-          <cylinder radius="0.007957385" length="0.030371133"/>
-        </geometry>
-      </collision>
-      <collision name="collision_index_post_sensor">
-        <origin xyz="0.00270223 0.014599754 0.001277816" rpy="1.307256699 -1.502358675 0.115027107"/>
-        <geometry>
-          <cylinder radius="0.007128498" length="0.014262123"/>
-        </geometry>
-      </collision>
-      <collision name="collision_index_tip">
-        <origin xyz="-0.010449275 0.059659205 0.000670571" rpy="-0.714037061 -1.367512941 1.09491086"/>
-        <geometry>
-          <sphere radius="0.006627175"/>
-        </geometry>
-      </collision>
-    </link>
-    <link name="little_fle">
-      <inertial>
-        <origin xyz="-0.00155 0.020800009 -3.5793e-05" rpy="0 0 0"/>
-        <mass value="0.0207"/>
-        <inertia ixx="7.686e-06" ixy="0" ixz="0" iyy="6.52e-07" iyz="0" izz="7.9e-06"/>
-      </inertial>
-      <visual >
-        <origin xyz="0.021798987 -0.079884358 -0.042128358" rpy="-0.088661931 -1.918641925 1.604480386"/>
-        <geometry>
-          <mesh filename="package://mia_hand_description/meshes/stl/little_finger.stl" scale="0.000999987 0.000999987 0.000999987"/>
-        </geometry>
-        <material name="BLACK"/>
-      </visual>
-      <visual >
-        <origin xyz="0.021798987 -0.079884358 -0.042128358" rpy="-0.088661931 -1.918641925 1.604480386"/>
-        <geometry>
-          <mesh filename="package://mia_hand_description/meshes/stl/little_tip.stl" scale="0.000999987 0.000999987 0.000999987"/>
-        </geometry>
-        <material name="WHITE"/>
-      </visual>
-      <collision name="collision_little_distal">
-        <origin xyz="-0.009071616 0.052363321 0.000405859" rpy="2.012047291 -1.547703743 0.014830198"/>
-        <geometry>
-          <cylinder radius="0.007603541" length="0.029933602"/>
-        </geometry>
-      </collision>
-      <collision name="collision_little_proximal">
-        <origin xyz="-0.001978738 0.027301736 -4.4674e-05" rpy="1.639323592 -1.540506959 -0.010816745"/>
-        <geometry>
-          <cylinder radius="0.007827824" length="0.030442052"/>
-        </geometry>
-      </collision>
-      <collision name="collision_little_tip">
-        <origin xyz="-0.016595591 0.064731956 -0.000363789" rpy="-1.135860085 -1.918640018 1.561329722"/>
-        <geometry>
-          <sphere radius="0.00484472"/>
-        </geometry>
-      </collision>
-    </link>
-    <link name="middle_fle">
-      <inertial>
-        <origin xyz="-6.3783e-05 0.006498255 -0.000197619" rpy="0 0 0"/>
-        <mass value="0.0123"/>
-        <inertia ixx="9.81e-07" ixy="0" ixz="0" iyy="2.03e-07" iyz="0" izz="9.33e-07"/>
-      </inertial>
-      <collision name="collision_middle_pre_sensor">
-        <origin xyz="5.4862e-05 0.02009861 0.000735957" rpy="1.572342396 -1.570796132 0"/>
-        <geometry>
-          <cylinder radius="0.006834491" length="0.01782351"/>
-        </geometry>
-      </collision>
-    </link>
-    <link name="middle_sensor">
-      <inertial>
-        <origin xyz="-0.003752992 0.025330022 7.9151e-05" rpy="0 0 0"/>
-        <mass value="0.0132"/>
-        <inertia ixx="4.326e-06" ixy="0" ixz="0" iyy="7.47e-07" iyz="0" izz="4.82e-06"/>
-      </inertial>
-      <visual>
-        <origin xyz="0.007670809 -0.12344341 -0.045150004" rpy="1.396263361 -1.570796371 0"/>
-        <geometry>
-          <mesh filename="package://mia_hand_description/meshes/stl/middle_finger.stl" scale="0.000999987 0.000999987 0.000999987"/>
-        </geometry>
-        <material name="BLACK"/>
-      </visual>
-      <visual >
-        <origin xyz="0.007670809 -0.12344341 -0.045150004" rpy="1.396263361 -1.570796371 0"/>
-        <geometry>
-          <mesh filename="package://mia_hand_description/meshes/stl/middle_tip.stl" scale="0.000999987 0.000999987 0.000999987"/>
-        </geometry>
-        <material name="WHITE"/>
-      </visual>
-      <collision name="collision_middle_distal">
-        <origin xyz="-0.008653791 0.039425109 0.000735376" rpy="2.091221809 -1.570796371 0"/>
-        <geometry>
-          <cylinder radius="0.008127632" length="0.038238756"/>
-        </geometry>
-      </collision>
-      <collision name="collision_middle_post_sensor">
-        <origin xyz="-0.000414368 0.010920909 0.000735376" rpy="1.572342396 -1.570796371 0"/>
-        <geometry>
-          <cylinder radius="0.00683449" length="0.011829435"/>
-        </geometry>
-      </collision>
-      <collision name="collision_middle_tip">
-        <origin xyz="-0.020539736 0.056403738 0.000735376" rpy="0.525144994 -1.570796371 0"/>
-        <geometry>
-          <sphere radius="0.005627529"/>
-        </geometry>
-      </collision>
-    </link>
-    <link name="palm">
-      <inertial>
-        <origin xyz="0.00268 0.067100011 -0.015999995" rpy="0 0 0"/>
-        <mass value="0.273999989"/>
-        <inertia ixx="0.000301" ixy="0" ixz="0" iyy="0.00013" iyz="0" izz="0.000343"/>
-      </inertial>
-      <visual >
-        <origin xyz="0.003035236 0.075372033 -0.025204176" rpy="-0.261799425 0 0"/>
-        <geometry>
-          <mesh filename="package://mia_hand_description/meshes/stl/dorsum_simple.stl" scale="0.076673768 0.104274787 0.076673768"/>
-        </geometry>
-        <material name="BLACK"/>
-      </visual>
-      <visual >
-        <origin xyz="0.003800225 0.065974504 -0.012054901" rpy="-0.261799335 0 0"/>
-        <geometry>
-          <mesh filename="package://mia_hand_description/meshes/stl/palm_simple.stl" scale="0.122026987 0.122026987 0.122026987"/>
-        </geometry>
-        <material name="BLACK"/>
-      </visual>
-      <visual >
-        <origin xyz="-0.039999999 0.015274569 -0.023892667" rpy="1.308997035 0 0"/>
-        <geometry>
-          <mesh filename="package://mia_hand_description/meshes/stl/wrist.stl" scale="0.000999999 0.000999999 0.000999999"/>
-        </geometry>
-        <material name="GREY"/>
-      </visual>
-      <collision name="collision_hand_distal">
-        <origin xyz="0.000396326 0.095129304 -0.021126958" rpy="-0.260977566 0.024364362 0.046443645"/>
-        <geometry>
-          <box size="0.072641067 0.047533765 0.033261035"/>
-        </geometry>
-      </collision>
-      <collision name="collision_hand_proximal">
-        <origin xyz="0.001288421 0.04622658 -0.005689064" rpy="-0.265261889 -0.179528236 0.101421639"/>
-        <geometry>
-          <box size="0.062414549 0.056382477 0.028578509"/>
-        </geometry>
-      </collision>
-    </link>
-    <!-- end effector -->
-    <link name="hand_ee_link" />
-    <joint name="palm_to_hand_ee_link" type="fixed">
-        <origin xyz="0 0.13 0.03" rpy="-0.65 0 0"/>
-      <parent link="palm"/>
-      <child link="hand_ee_link"/>
-    </joint>
-    <link name="ring_fle">
-      <inertial>
-        <origin xyz="-0.001120002 0.026399991 0.000203993" rpy="0 0 0"/>
-        <mass value="0.0263"/>
-        <inertia ixx="1.577e-05" ixy="0" ixz="0" iyy="9.02e-07" iyz="0" izz="1.61e-05"/>
-      </inertial>
-      <visual >
-        <origin xyz="0.01104607 -0.090066954 -0.043558836" rpy="1.65e-07 -1.745330095 1.413716316"/>
-        <geometry>
-          <mesh filename="package://mia_hand_description/meshes/stl/ring_finger.stl" scale="0.000999987 0.000999987 0.000999987"/>
-        </geometry>
-        <material name="BLACK"/>
-      </visual>
-      <visual >
-        <origin xyz="0.01104607 -0.090066954 -0.043558836" rpy="1.65e-07 -1.745330095 1.413716316"/>
-        <geometry>
-          <mesh filename="package://mia_hand_description/meshes/stl/ring_tip.stl" scale="0.000999987 0.000999987 0.000999987"/>
-        </geometry>
-        <material name="WHITE"/>
-      </visual>
-      <collision name="collision_ring_distal">
-        <origin xyz="-0.008521391 0.063275322 0.000219088" rpy="2.099160433 -1.578026533 0.020510485"/>
-        <geometry>
-          <cylinder radius="0.00760354" length="0.029933617"/>
-        </geometry>
-      </collision>
-      <collision name="collision_ring_proximal">
-        <origin xyz="0.001186912 0.028925091 0.000219103" rpy="1.570796132 -1.570796251 0"/>
-        <geometry>
-          <cylinder radius="0.007827824" length="0.03682825"/>
-        </geometry>
-      </collision>
-      <collision name="collision_ring_tip">
-        <origin xyz="-0.018231211 0.076642096 -0.000189718" rpy="-1.047197104 -1.745329261 1.570796132"/>
-        <geometry>
-          <sphere radius="0.004873112"/>
-        </geometry>
-      </collision>
-    </link>
-    <link name="thumb_fle">
-      <inertial>
-        <origin xyz="0.012771533 0.029501937 0.000170548" rpy="0 0 0"/>
-        <mass value="0.0592"/>
-        <inertia ixx="4e-05" ixy="1.3e-08" ixz="0" iyy="3e-06" iyz="4e-09" izz="4.1e-05"/>
-      </inertial>
-      <visual >
-        <origin xyz="-0.003567816 -0.07197547 0.054485805" rpy="0.62849319 1.087863922 0.258483142"/>
-        <geometry>
-          <mesh filename="package://mia_hand_description/meshes/stl/thumb_cover.stl" scale="0.000999988 0.000999987 0.000999987"/>
-        </geometry>
-        <material name="WHITE"/>
-      </visual>
-      <visual >
-        <origin xyz="-0.003567816 -0.07197547 0.054485805" rpy="0.62849319 1.087863922 0.258483142"/>
-        <geometry>
-          <mesh filename="package://mia_hand_description/meshes/stl/thumb_frame.stl" scale="0.000999988 0.000999987 0.000999987"/>
-        </geometry>
-        <material name="GREY"/>
-      </visual>
-      <collision name="collision_thumb_distal">
-        <origin xyz="0.015668914 0.047384627 0.001403906" rpy="1.470562816 0.195132375 -0.047180746"/>
-        <geometry>
-          <cylinder radius="0.011694114" length="0.055018328"/>
-        </geometry>
-      </collision>
-      <collision name="collision_thumb_proximal">
-        <origin xyz="0.015613321 0.032607533 6.2179e-05" rpy="1.543844342 0.23866643 -0.080058314"/>
-        <geometry>
-          <cylinder radius="0.012714386" length="0.059818495"/>
-        </geometry>
-      </collision>
-      <collision name="collision_thumb_tip">
-        <origin xyz="0.015702201 0.069964014 -0.00075977" rpy="-0.3828291 0.583412647 0.648222387"/>
-        <geometry>
-          <sphere radius="0.010514786"/>
-        </geometry>
-      </collision>
-    </link>
-    <link name="thumb_opp">
-      <inertial>
-        <origin xyz="0.00026099 0.007620003 0.001220003" rpy="0 0 0"/>
-        <mass value="0.013"/>
-        <inertia ixx="1.12e-06" ixy="0" ixz="0" iyy="1.2e-07" iyz="0" izz="1.15e-06"/>
-      </inertial>
-      <visual >
-        <origin xyz="-0.054523792 -0.04869514 0.027307283" rpy="-0.128456295 -0.364075422 0.324456483"/>
-        <geometry>
-          <mesh filename="package://mia_hand_description/meshes/stl/thumb_metacarpus.stl" scale="0.000999987 0.000999987 0.000999987"/>
-        </geometry>
-        <material name="GREY"/>
-      </visual>
-    </link>
-    <link name="thumb_sensor">
-      <inertial>
-        <origin xyz="-1.5e-08 -9e-09 -4e-09" rpy="0 0 0"/>
-        <mass value="0.000643"/>
-        <inertia ixx="1.5e-08" ixy="0" ixz="0" iyy="8e-09" iyz="0" izz="1.5e-08"/>
-      </inertial>
-    </link>
-    <joint name="j_index_fle" type="revolute">
-      <origin xyz="0.026305504 0.11021702 -0.021520771" rpy="-0.596919358 1.415553689 -0.749806523"/>
-      <parent link="palm"/>
-      <child link="index_fle"/>
-      <dynamics damping="0.1"/>
-      <axis xyz="-6e-08 1.7e-08 0.99999994"/>
-      <limit lower="-1.399999976" upper="1.399999976" effort="1.75" velocity="3.140000105"/>
-    </joint>
-    <joint name="j_index_sensor" type="fixed">
-      <origin xyz="-0.000399255 0.024237007 -0.000183955" rpy="0.000630725 -0.000209123 0.172082633"/>
-      <parent link="index_fle"/>
-      <child link="index_sensor"/>
-    </joint>
-    <joint name="j_little_fle" type="revolute">
-      <origin xyz="-0.027859999 0.107325219 -0.020605115" rpy="1.278342605 1.775918841 1.627186179"/>
-      <parent link="palm"/>
-      <child link="little_fle"/>
-      <dynamics damping="0.1"/>
-      <axis xyz="-6e-08 1.7e-08 1.0"/>
-      <limit lower="0" upper="1.396260023" effort="1.75" velocity="3.140000105"/>
-      <mimic joint="j_mrl_fle" multiplier="1" offset="0" /> <!-- to be manually added for Rviz -->
-    </joint>
-    <joint name="j_mrl_fle" type="revolute">
-      <origin xyz="0.00514942 0.113555029 -0.024345273" rpy="-1.570794106 1.483529925 -1.570793986"/>
-      <parent link="palm"/>
-      <child link="middle_fle"/>
-      <dynamics damping="0.1"/>
-      <axis xyz="-6e-08 1.7e-08 0.99999994"/>
-      <limit lower="0" upper="1.396260023" effort="1.75" velocity="3.140000105"/>
-    </joint>
-    <joint name="j_middle_sensor" type="fixed">
-      <origin xyz="0.000444004 0.025497464 5.81e-07" rpy="1.8e-08 2.07e-07 -3e-08"/>
-      <parent link="middle_fle"/>
-      <child link="middle_sensor"/>
-    </joint>
-    <joint name="j_ring_fle" type="revolute">
-      <origin xyz="-0.012250358 0.112028912 -0.023936352" rpy="1.150808096 1.681244493 1.321779966"/>
-      <parent link="palm"/>
-      <child link="ring_fle"/>
-      <dynamics damping="0.1"/>
-      <axis xyz="-6e-08 1.7e-08 1.0"/>
-      <limit lower="0" upper="1.396260023" effort="1.75" velocity="3.140000105"/>
-      <mimic joint="j_mrl_fle" multiplier="1" offset="0" /> <!-- to be manually added for Rviz -->
-    </joint>
-    <joint name="j_thumb_fle" type="revolute">
-      <origin xyz="-2.7426e-05 -1.0543e-05 -0.008989788" rpy="-1.570910335 0.438224047 1.570665002"/>
-      <parent link="thumb_sensor"/>
-      <child link="thumb_fle"/>
-      <dynamics damping="0.1"/>
-      <axis xyz="-6e-08 1.7e-08 1.0"/>
-      <limit lower="0" upper="1.134500027" effort="3.5" velocity="1.570000052"/>
-    </joint>
-    <joint name="j_thumb_opp" type="revolute">
-      <origin xyz="0.013073999 0.068108179 -0.001949422" rpy="1.43719089 0.369162768 0.318591952"/>
-      <parent link="palm"/>
-      <child link="thumb_opp"/>
-      <dynamics damping="0.2"/>
-      <axis xyz="-6e-08 1.7e-08 1.0"/>
-      <limit lower="-0.628318548" upper="0" effort="3.5" velocity="4.0"/>
-    </joint>
-    <joint name="j_thumb_sensor" type="fixed">
-      <origin xyz="-5.942e-06 0.008997655 2.453e-06" rpy="1.570796371 1.01e-07 -1.19e-07"/>
-      <parent link="thumb_opp"/>
-      <child link="thumb_sensor"/>
-    </joint>
+<!-- model version="4.4.2"-->
+<robot name="mia_hand" xmlns:xacro="http://wiki.ros.org/xacro" xmlns:body="http://playerstage.sourceforge.net/gazebo/xmlschema/#body" xmlns:controller="http://playerstage.sourceforge.net/gazebo/xmlschema/#controller" xmlns:geom="http://playerstage.sourceforge.net/gazebo/xmlschema/#geom" xmlns:interface="http://playerstage.sourceforge.net/gazebo/xmlschema/#interface" xmlns:joint="http://playerstage.sourceforge.net/gazebo/xmlschema/#slider" xmlns:sensor="http://playerstage.sourceforge.net/gazebo/xmlschema/#sensor">
+  <xacro:macro name="mia_hand_robot" params="
+    joint_limits_parameters_file:= '$(find mia_hand_description)/calibration/joint_limits_default.yaml' " >
+      <!-- Include the macro to read yaml File-->
+      <xacro:include filename="$(find mia_hand_description)/urdf/inc/mia_hand_common.xacro" />
+      <!-- Load configuration data from the provided .yaml files -->
+      <xacro:read_model_data
+        joint_limits_parameters_file="${joint_limits_parameters_file}"/>
+      <!-- URDF of the hand using loaded data -->
+      <link name="index_fle">
+        <inertial>
+          <origin xyz="0 0 0" rpy="0 0 0"/>
+          <mass value="0.01113"/>
+          <inertia ixx="1.40e-06" ixy="1.58e-08" ixz="0" iyy="1.97e-07" iyz="2.27e-10" izz="1.36e-06"/>
+        </inertial>
+        <collision name="collision_index_pre_sensor">
+          <origin xyz="0.000159719 0.023606986 0.001508433" rpy="1.611356378 -1.479902387 -0.009164433"/>
+          <geometry>
+            <cylinder radius="0.007128498" length="0.016970539"/>
+          </geometry>
+        </collision>
+      </link>
+    	<link name="index_sensor">
+        <inertial>
+          <origin xyz="0 0 0" rpy="0 0 0"/>
+          <mass value="0.01765"/>
+          <inertia ixx="2.07e-05" ixy="4.28e-06" ixz="7.05e-09" iyy="1.71e-06" iyz="-5.40e-09" izz="2.19e-05"/>
+        </inertial>
+        <visual >
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