Commit message: Use URDF

File: hand_embodiment/model/mia_hand_ros_pkgs/mia_hand_description/urdf/mia_hand.urdf (robot description, URDF)
Before this commit: robot mia_hand, 10 links, 9 joints
Links:
- added link hand_ee_link, mass 0.0
- link index_fle: mass 0.0113 -> 0.01113
- link index_sensor: mass 0.0132 -> 0.01765
- link middle_fle: mass 0.0123 -> 0.0121
- link middle_sensor: mass 0.0132 -> 0.0177
- link thumb_fle: geometry collision cylinder length=0.055018328 radius=0.011694114; collision cylinder length=0.059818495 radius=0.012714386
Joints:
- added joint palm_to_hand_ee_link: type fixed, parent palm, child hand_ee_link, origin xyz=0 0.13 0.03 rpy=-0.65 0 0
- joint j_index_fle: axis 0 0 1.0 -> -6e-08 1.7e-08 0.99999994
- joint j_little_fle: axis 0 0 1.0 -> -6e-08 1.7e-08 1.0
- joint j_mrl_fle: axis 0 0 1.0 -> -6e-08 1.7e-08 0.99999994
- joint j_ring_fle: axis 0 0 1.0 -> -6e-08 1.7e-08 1.0
- joint j_thumb_fle: axis 0 0 1.0 -> -6e-08 1.7e-08 1.0; limit lower=0.0 upper=1.134500027 effort=3.5 velocity=1.570000052 -> lower=0 upper=1.134500027 effort=3.5 velocity=1.570000052; origin xyz=-2.7433e-05 0.008989773 -1.0513e-05 rpy=-1.570600271 -1.132572651 1.570515633 -> xyz=-2.7426e-05 -1.0543e-05 -0.008989788 rpy=-1.570910335 0.438224047 1.570665002
- joint j_thumb_opp: axis 0 0 1.0 -> -6e-08 1.7e-08 1.0
- joint j_thumb_sensor: origin xyz=-5.942e-06 0.008997655 2.453e-06 rpy=-1.56e-07 4.8e-08 -6e-08 -> xyz=-5.942e-06 0.008997655 2.453e-06 rpy=1.570796371 1.01e-07 -1.19e-07
